Commit message: Renamed drive_bot to my_robot

File: my_robot/urdf/my_robot.xacro (robot description, xacro)
@@ -3,5 +3,5 @@
      Commit Version: 1.6.0-4-g7f85cfe  Build Version: 1.6.7995.38578
      For more information, please see http://wiki.ros.org/sw_urdf_exporter -->
-<robot name="drive_bot" xmlns:xacro="http://www.ros.org/wiki/xacro">
+<robot name="my_robot" xmlns:xacro="http://www.ros.org/wiki/xacro">
   <link name="base_link">
     <!-- <pose>0 0 0.04 0 0 0</pose> -->
@@ -14,5 +14,5 @@
       <origin xyz="0 0 0" rpy="0 0 0" />
       <geometry>
-        <mesh filename="package://drive_bot/meshes/base_link.STL" />
+        <mesh filename="package://my_robot/meshes/base_link.STL" />
       </geometry>
       <material name="">
@@ -23,5 +23,5 @@
       <origin xyz="0 0 0" rpy="0 0 0" />
       <geometry>
-        <mesh filename="package://drive_bot/meshes/base_link.STL" />
+        <mesh filename="package://my_robot/meshes/base_link.STL" />
       </geometry>
     </collision>
@@ -36,5 +36,5 @@
       <origin xyz="-0.04 -0.03 -0.03" rpy="0 0 0" />
       <geometry>
-        <mesh filename="package://drive_bot/meshes/left_wheel.STL" />
+        <mesh filename="package://my_robot/meshes/left_wheel.STL" />
       </geometry>
       <material name="">
@@ -45,5 +45,5 @@
       <origin xyz="-0.04 -0.03 -0.03" rpy="0 0 0" />
       <geometry>
-        <mesh filename="package://drive_bot/meshes/left_wheel.STL" />
+        <mesh filename="package://my_robot/meshes/left_wheel.STL" />
       </geometry>
     </collision>
@@ -58,5 +58,5 @@
       <origin xyz="-0.04 -0.03 0.03" rpy="0 0 0" />
       <geometry>
-        <mesh filename="package://drive_bot/meshes/right_wheel.STL" />
+        <mesh filename="package://my_robot/meshes/right_wheel.STL" />
       </geometry>
       <material name="">
@@ -67,5 +67,5 @@
       <origin xyz="-0.04 -0.03 0.03" rpy="0 0 0" />
       <geometry>
-        <mesh filename="package://drive_bot/meshes/right_wheel.STL" />
+        <mesh filename="package://my_robot/meshes/right_wheel.STL" />
       </geometry>
     </collision>
@@ -158,4 +158,4 @@
     </material>
   </gazebo>
-  <xacro:include filename="$(find drive_bot)/urdf/drive_bot.gazebo" />
+  <xacro:include filename="$(find my_robot)/urdf/my_robot.gazebo" />
 </robot>
